File: 1_ega/3_esquematico_pcb/Esquematico_EGA.kicad_pcb (KiCad board)
At the start: 2 copper layers, 100 x 100 mm, 66 parts, among them J1 ±5V, J2 UART, J3 Encoder, J4 CP2102, J5 OUT, J6 IN, J7 DDS, J8 Conn_01x14, J9 Conn_01x14, Q1 2N7000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

Commit message: actualizar esquemático y layout PCB
Parts:
- moved J3 24.6 mm to (109.7, 121.8)
- moved TP8 21.3 mm to (161.3, 139.3)
- moved TP6 19.4 mm to (117.3, 120.0)
- moved SW1 17.4 mm to (96.3, 133.0), turned to 180 degrees
- moved TP3 15.2 mm to (129.3, 128.0)
- moved TP4 15.0 mm to (129.3, 120.0)
- moved TP9 13.2 mm to (137.3, 138.3)
- moved C1 13.2 mm to (163.3, 76.0)
- moved C10 13.2 mm to (163.3, 97.2)
- moved C11 13.2 mm to (147.3, 127.3)
- moved C12 13.2 mm to (147.3, 99.7)
- moved C2 13.2 mm to (144.8, 83.6)
- moved C3 13.2 mm to (168.3, 61.3)
- moved C4 13.2 mm to (155.5, 61.3)
- moved C5 13.2 mm to (140.3, 53.8)
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Routing:
- net GND: track 530.4 -> 609.0 mm
- net +3.3V: track 173.8 -> 152.5 mm
- net /ENC_SW: track 27.9 -> 13.4 mm
- net /ENC_CLK: track 27.9 -> 13.4 mm
- net /ENC_DT: track 27.9 -> 13.4 mm
- net /BTN_2: track 30.4 -> 43.5 mm
- net /BTN_1: track 20.7 -> 28.7 mm
- net /Reset_Vin: track 39.6 -> 44.8 mm
- net +5V: track 305.5 -> 310.7 mm
- net /Reset_Vout: track 49.1 -> 44.6 mm
- net /Vin_pico: track 50.5 -> 48.9 mm
- net /Vout_pico: track 61.9 -> 60.5 mm

Commit message: actualización PCB y esquemático
Parts:
- TP7: value Vin -> DDS_out
Changed lines of the file:
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@@
 		(filling no)
 		(pcbplotparams
-			(layerselection 0x00000000_00000000_55555555_55555554)
+			(layerselection 0x00000000_00000000_5555555d_55555550)
 			(plot_on_all_layers_selection 0x00000000_00000000_00000000_02000000)
 			(disableapertmacros no)
@@
 			)
 		)
-		(property "Value" "Vin"
+		(property "Value" "DDS_out"
 			(at 0 2.38 0)
 			(layer "F.Fab")

Commit message: Cambiar operacional por el TL072
Parts:
- U1, U2, U3: value OPA2134 -> TL072
Changed lines of the file:
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@@
 		(filling no)
 		(pcbplotparams
-			(layerselection 0x00000000_00000000_5555555d_55555550)
+			(layerselection 0x00000000_00000000_55555555_55555554)
 			(plot_on_all_layers_selection 0x00000000_00000000_00000000_02000000)
 			(disableapertmacros no)
@@
 			)
 		)
-		(property "Value" "OPA2134"
+		(property "Value" "TL072"
 			(at 3.81 -2.42 0)
 			(layer "F.Fab")
@@
 			)
 		)
-		(property "Value" "OPA2134"
+		(property "Value" "TL072"
 			(at 3.81 -2.466996 0)
 			(layer "F.Fab")
@@
 			)
 		)
-		(property "Value" "OPA2134"
+		(property "Value" "TL072"
 			(at 3.81 9.95 0)
 			(layer "F.Fab")
